File: motion_detect.sch (EAGLE design)
At the start: 81 parts, among them CON1 PINHEAD_1X02-2.54, CON2 PINHEAD_1X01-2.54, CON3 PINHEAD_1X08-2.54, CON4 PINHEAD_1X05-2.54, CON5 PINHEAD_1X01-2.54, CON6 USB-2, IC1 5.0, IC2 LTC4054, IC3 3.3, IC4 ATMEGA168-TQFP32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

Commit message: some minor BOM fixes
Parts:
- LED1: ASSEMBLY SPECIAL -> (none); BOM OPTIONAL -> (none); COLOR RED -> BLUE; LINK http://www.zip-2002.ru/osveshchenie_i_indikatsiya/svetodiod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 -> (none)
- LED2: COLOR GREEN -> BLUE
- LED5: ASSEMBLY SPECIAL -> (none); BOM OPTIONAL -> (none); LINK http://www.zip-2002.ru/osveshchenie_i_indikatsiya/svetodiod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 -> (none)
Changed lines of the file:
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@@
 <part name="FRAME1" library="frames" deviceset="A4L-LOC" device=""/>
 <part name="LED2" library="rc" deviceset="LED" device="-0603">
-<attribute name="COLOR" value="GREEN"/>
+<attribute name="COLOR" value="BLUE"/>
 </part>
 <part name="R2" library="rc" deviceset="R" device="-0603" value="1K"/>
@@
 <part name="+P24" library="supply_symbols" deviceset="VBAT" device=""/>
 <part name="LED5" library="dp_devices" deviceset="LED" device="-3MM">
-<attribute name="ASSEMBLY" value="SPECIAL"/>
-<attribute name="BOM" value="OPTIONAL"/>
 <attribute name="COLOR" value="RED"/>
-<attribute name="LINK" value="http://www.zip-2002.ru/osveshchenie_i_indikatsiya/svetodiody/86349/1x3x4_red_50_mcd_2,1v/"/>
 </part>
 <part name="LED1" library="dp_devices" deviceset="LED" device="-3MM">
-<attribute name="ASSEMBLY" value="SPECIAL"/>
-<attribute name="BOM" value="OPTIONAL"/>
-<attribute name="COLOR" value="RED"/>
-<attribute name="LINK" value="http://www.zip-2002.ru/osveshchenie_i_indikatsiya/svetodiody/86349/1x3x4_red_50_mcd_2,1v/"/>
+<attribute name="COLOR" value="BLUE"/>
 </part>
 <part name="R20" library="rc" deviceset="R" device="-0603" value="4K7"/>
@@
 <instance part="+P24" gate="G$1" x="160.02" y="170.18"/>
 <instance part="LED5" gate="LED" x="154.94" y="114.3">
-<attribute name="BOM" x="154.94" y="114.3" size="1.778" layer="96" display="off"/>
 <attribute name="COLOR" x="154.94" y="114.3" size="1.778" layer="96" display="off"/>
-<attribute name="LINK" x="154.94" y="114.3" size="1.778" layer="96" display="off"/>
 </instance>
 <instance part="LED1" gate="LED" x="167.64" y="114.3">
-<attribute name="BOM" x="167.64" y="114.3" size="1.778" layer="96" display="off"/>
 <attribute name="COLOR" x="167.64" y="114.3" size="1.778" layer="96" display="off"/>
-<attribute name="LINK" x="167.64" y="114.3" size="1.778" layer="96" display="off"/>
 </instance>
 <instance part="R20" gate="G$1" x="71.12" y="134.62" rot="R270"/>

Commit message: new version
Parts:
- removed LED2, LED4: LED-0603, rc:LED-0603
- removed Z1: 8MHz, led_matrix_master_lib:CRYSTAL-3.2X2.5-4P
- SW1: value TACT_SWITCH -> TACT_SWITCH-TC-206; device motion_detect_masterlib:TACT_SWITCH -> motion_detect_masterlib:TACT_SWITCH-TC-206
Connections:
- removed net CHRG_LED: IC2.CHRG
- removed net N$19: MODULE2.PIO1, R3.2
- net A0: now also R1.2, R18.1; no longer R11.1
- net A7: now also CON3.6; no longer CON3.5
- net D2: now also R11.1; no longer CON3.6
- net D3: now also SW1.1; no longer R1.2, R18.1
- net D4: now also MODULE2.UART_RX; no longer SW1.2
- net D8: now also MODULE2.PIO1, R3.2; no longer MODULE2.UART_RX
- net GND: now also SW1.2; no longer SW1.1
- net MISO: now also CON3.3; no longer CON3.2
- net MOSI: now also CON3.5; no longer CON3.4
- net N$12: no longer LED4.C
- net N$2: no longer LED2.C
- net N$6: no longer Z1.2
- net N$8: no longer Z1.1
- net SCK: now also CON3.4; no longer CON3.3
- net SUP: no longer LED4.A
- net VDD_3V3: no longer LED2.A
- net VDD_5V: now also CON3.2
Other:
- moved on the sheet: LED1, LED5, R1, R18, R20, SW1

Commit message: update
Parts:
- added CON7: PINHEAD_1X03-2.54, pinhead:PINHEAD_1X03-2.54
Connections:
- new net N$14: CON7.2, CON7.3
- net D4: now also MODULE2.PIO1, R3.2; no longer MODULE2.UART_RX
- net D8: now also MODULE2.UART_RX; no longer MODULE2.PIO1, R3.2
Changed lines of the file:
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@@
 <part name="+P1" library="supply_symbols" deviceset="3.3V" device=""/>
 <part name="+P26" library="supply_symbols" deviceset="5V" device=""/>
+<part name="CON7" library="pinhead" deviceset="PINHEAD_1X03" device="-2.54"/>
 </parts>
 <sheets>
@@
 <instance part="+P1" gate="G$1" x="71.12" y="139.7"/>
 <instance part="+P26" gate="G$1" x="25.4" y="127" rot="R270"/>
+<instance part="CON7" gate="G$1" x="248.92" y="147.32" rot="R180"/>
 </instances>
 <busses>
@@
 </segment>
 <segment>
+<pinref part="MODULE2" gate="G$1" pin="UART_RX"/>
+<wire x1="195.58" y1="81.28" x2="193.04" y2="81.28" width="0.1524" layer="91"/>
+<label x="193.04" y="81.28" size="1.27" layer="95" rot="R180" xref="yes"/>
+</segment>
+</net>
+<net name="A3" class="0">
+<segment>
+<pinref part="IC4" gate="G$1" pin="PC3"/>
+<wire x1="106.68" y1="137.16" x2="106.68" y2="139.7" width="0.1524" layer="91"/>
+<label x="106.68" y="139.7" size="1.27" layer="95" rot="R90" xref="yes"/>
+</segment>
+<segment>
+<pinref part="Q1" gate="G$1" pin="G"/>
+<wire x1="195.58" y1="109.22" x2="190.5" y2="109.22" width="0.1524" layer="91"/>
+<label x="187.96" y="109.22" size="1.27" layer="95" rot="R180" xref="yes"/>
+<pinref part="R15" gate="G$1" pin="2"/>
+<wire x1="190.5" y1="109.22" x2="187.96" y2="109.22" width="0.1524" layer="91"/>
+<wire x1="190.5" y1="111.76" x2="190.5" y2="109.22" width="0.1524" layer="91"/>
+<junction x="190.5" y="109.22"/>
+</segment>
+</net>
+<net name="A2" class="0">
+<segment>
+<pinref part="IC4" gate="G$1" pin="PC2"/>
+<wire x1="109.22" y1="137.16" x2="109.22" y2="139.7" width="0.1524" layer="91"/>
+<label x="109.22" y="139.7" size="1.27" layer="95" rot="R90" xref="yes"/>
+</segment>
+<segment>
+<pinref part="CON3" gate="G$1" pin="7"/>
+<wire x1="15.24" y1="139.7" x2="20.32" y2="139.7" width="0.1524" layer="91"/>
+<label x="20.32" y="139.7" size="1.27" layer="95" xref="yes"/>
+</segment>
+</net>
+<net name="A1" class="0">
+<segment>
+<pinref part="IC4" gate="G$1" pin="PC1"/>
+<wire x1="119.38" y1="127" x2="121.92" y2="127" width="0.1524" layer="91"/>
+<label x="121.92" y="127" size="1.27" layer="95" xref="yes"/>
+</segment>
+<segment>
+<pinref part="MODULE3" gate="G$1" pin="SET"/>
+<wire x1="213.36" y1="114.3" x2="210.82" y2="114.3" width="0.1524" layer="91"/>
+<label x="210.82" y="114.3" size="1.27" layer="95" rot="R180" xref="yes"/>
+</segment>
+</net>
+<net name="A0" class="0">
+<segment>
+<pinref part="IC4" gate="G$1" pin="PC0"/>
+<wire x1="119.38" y1="124.46" x2="121.92" y2="124.46" width="0.1524" layer="91"/>
+<label x="121.92" y="124.46" size="1.27" layer="95" xref="yes"/>
+</segment>
+<segment>
+<pinref part="R18" gate="G$1" pin="1"/>
+<pinref part="R1" gate="G$1" pin="2"/>
+<wire x1="45.72" y1="132.08" x2="45.72" y2="129.54" width="0.1524" layer="91"/>
+<wire x1="45.72" y1="129.54" x2="45.72" y2="127" width="0.1524" layer="91"/>
+<wire x1="45.72" y1="129.54" x2="48.26" y2="129.54" width="0.1524" layer="91"/>
+<junction x="45.72" y="129.54"/>
+<label x="48.26" y="129.54" size="1.27" layer="95" xref="yes"/>
+</segment>
+</net>
+<net name="D2" class="0">
+<segment>
+<pinref part="IC4" gate="G$1" pin="PD2"/>
+<wire x1="91.44" y1="137.16" x2="91.44" y2="139.7" width="0.1524" layer="91"/>
+<wire x1="91.44" y1="139.7" x2="88.9" y2="139.7" width="0.1524" layer="91"/>
+<label x="88.9" y="139.7" size="1.27" layer="95" rot="R180" xref="yes"/>
+</segment>
+<segment>
+<wire x1="218.44" y1="157.48" x2="215.9" y2="157.48" width="0.1524" layer="91"/>
+<label x="215.9" y="157.48" size="1.27" layer="95" rot="R180" xref="yes"/>
+<pinref part="R11" gate="G$1" pin="1"/>
+</segment>
+</net>
+<net name="D4" class="0">
+<segment>
+<pinref part="IC4" gate="G$1" pin="PD4"/>
+<wire x1="81.28" y1="124.46" x2="71.12" y2="124.46" width="0.1524" layer="91"/>
+<label x="68.58" y="124.46" size="1.27" layer="95" rot="R180" xref="yes"/>
+<pinref part="R20" gate="G$1" pin="2"/>
+<wire x1="71.12" y1="124.46" x2="68.58" y2="124.46" width="0.1524" layer="91"/>
+<wire x1="71.12" y1="127" x2="71.12" y2="124.46" width="0.1524" layer="91"/>
+<junction x="71.12" y="124.46"/>
+</segment>
+<segment>
 <pinref part="MODULE2" gate="G$1" pin="PIO1"/>
 <wire x1="238.76" y1="58.42" x2="248.92" y2="58.42" width="0.1524" layer="91"/>
@@
 <junction x="248.92" y="58.42"/>
 <label x="248.92" y="60.96" size="1.27" layer="95" rot="R90" xref="yes"/>
-</segment>
-</net>
-<net name="A3" class="0">
-<segment>
-<pinref part="IC4" gate="G$1" pin="PC3"/>
-<wire x1="106.68" y1="137.16" x2="106.68" y2="139.7" width="0.1524" layer="91"/>
-<label x="106.68" y="139.7" size="1.27" layer="95" rot="R90" xref="yes"/>
-</segment>
-<segment>
-<pinref part="Q1" gate="G$1" pin="G"/>
-<wire x1="195.58" y1="109.22" x2="190.5" y2="109.22" width="0.1524" layer="91"/>
-<label x="187.96" y="109.22" size="1.27" layer="95" rot="R180" xref="yes"/>
-<pinref part="R15" gate="G$1" pin="2"/>
-<wire x1="190.5" y1="109.22" x2="187.96" y2="109.22" width="0.1524" layer="91"/>
-<wire x1="190.5" y1="111.76" x2="190.5" y2="109.22" width="0.1524" layer="91"/>
-<junction x="190.5" y="109.22"/>
-</segment>
-</net>
-<net name="A2" class="0">
-<segment>
-<pinref part="IC4" gate="G$1" pin="PC2"/>
-<wire x1="109.22" y1="137.16" x2="109.22" y2="139.7" width="0.1524" layer="91"/>
-<label x="109.22" y="139.7" size="1.27" layer="95" rot="R90" xref="yes"/>
-</segment>
-<segment>
-<pinref part="CON3" gate="G$1" pin="7"/>
-<wire x1="15.24" y1="139.7" x2="20.32" y2="139.7" width="0.1524" layer="91"/>
-<label x="20.32" y="139.7" size="1.27" layer="95" xref="yes"/>
-</segment>
-</net>
-<net name="A1" class="0">
-<segment>
-<pinref part="IC4" gate="G$1" pin="PC1"/>
-<wire x1="119.38" y1="127" x2="121.92" y2="127" width="0.1524" layer="91"/>
-<label x="121.92" y="127" size="1.27" layer="95" xref="yes"/>
-</segment>
-<segment>
-<pinref part="MODULE3" gate="G$1" pin="SET"/>
-<wire x1="213.36" y1="114.3" x2="210.82" y2="114.3" width="0.1524" layer="91"/>
-<label x="210.82" y="114.3" size="1.27" layer="95" rot="R180" xref="yes"/>
-</segment>
-</net>
-<net name="A0" class="0">
-<segment>
-<pinref part="IC4" gate="G$1" pin="PC0"/>
-<wire x1="119.38" y1="124.46" x2="121.92" y2="124.46" width="0.1524" layer="91"/>
-<label x="121.92" y="124.46" size="1.27" layer="95" xref="yes"/>
-</segment>
-<segment>
-<pinref part="R18" gate="G$1" pin="1"/>
-<pinref part="R1" gate="G$1" pin="2"/>
-<wire x1="45.72" y1="132.08" x2="45.72" y2="129.54" width="0.1524" layer="91"/>
-<wire x1="45.72" y1="129.54" x2="45.72" y2="127" width="0.1524" layer="91"/>
-<wire x1="45.72" y1="129.54" x2="48.26" y2="129.54" width="0.1524" layer="91"/>
-<junction x="45.72" y="129.54"/>
-<label x="48.26" y="129.54" size="1.27" layer="95" xref="yes"/>
-</segment>
-</net>
-<net name="D2" class="0">
-<segment>
-<pinref part="IC4" gate="G$1" pin="PD2"/>
-<wire x1="91.44" y1="137.16" x2="91.44" y2="139.7" width="0.1524" layer="91"/>
-<wire x1="91.44" y1="139.7" x2="88.9" y2="139.7" width="0.1524" layer="91"/>
-<label x="88.9" y="139.7" size="1.27" layer="95" rot="R180" xref="yes"/>
-</segment>
-<segment>
-<wire x1="218.44" y1="157.48" x2="215.9" y2="157.48" width="0.1524" layer="91"/>
-<label x="215.9" y="157.48" size="1.27" layer="95" rot="R180" xref="yes"/>
-<pinref part="R11" gate="G$1" pin="1"/>
-</segment>
-</net>
-<net name="D4" class="0">
-<segment>
-<pinref part="IC4" gate="G$1" pin="PD4"/>
-<wire x1="81.28" y1="124.46" x2="71.12" y2="124.46" width="0.1524" layer="91"/>
-<label x="68.58" y="124.46" size="1.27" layer="95" rot="R180" xref="yes"/>
-<pinref part="R20" gate="G$1" pin="2"/>
-<wire x1="71.12" y1="124.46" x2="68.58" y2="124.46" width="0.1524" layer="91"/>
-<wire x1="71.12" y1="127" x2="71.12" y2="124.46" width="0.1524" layer="91"/>
-<junction x="71.12" y="124.46"/>
-</segment>
-<segment>
-<pinref part="MODULE2" gate="G$1" pin="UART_RX"/>
-<wire x1="195.58" y1="81.28" x2="193.04" y2="81.28" width="0.1524" layer="91"/>
-<label x="193.04" y="81.28" size="1.27" layer="95" rot="R180" xref="yes"/>
 </segment>
 </net>
@@
 </segment>
 </net>
+<net name="N$14" class="0">
+<segment>
+<pinref part="CON7" gate="G$1" pin="2"/>
+<wire x1="241.3" y1="142.24" x2="238.76" y2="142.24" width="0.1524" layer="91"/>
+<wire x1="238.76" y1="142.24" x2="238.76" y2="139.7" width="0.1524" layer="91"/>
+<pinref part="CON7" gate="G$1" pin="3"/>
+<wire x1="238.76" y1="139.7" x2="241.3" y2="139.7" width="0.1524" layer="91"/>
+</segment>
+</net>

Commit message: -update
Parts:
- added Q5: IRLML2502-SOT23, motion_detect_masterlib:IRLML2502-SOT23
- added R21, R24: 24R, rc:R-R1206
- added R22, R23: 4K7, rc:R-0603
- R20: ASSY (none) -> DNM
- renumbered Z1_1 to Z1
Connections:
- new net N$26: Q5.D, R21.1, R24.1
- net A2: now also IC1.CE; no longer CON3.7
- net D10: now also Q5.G, R23.1; no longer IC1.CE
- net D3: now also R22.2
- net GND: now also CON3.7, Q5.S, R23.2
- net SUP: now also R21.2, R24.2
- net VDD_3V3: now also R22.1
Other:
- moved on the sheet: SW1
Changed lines of the file:
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@@
 <part name="+P23" library="supply_symbols" deviceset="5V" device=""/>
 <part name="R19" library="rc" deviceset="R" device="-0603" value="1K"/>
-<part name="Z1_1" library="ExitControl_v2_master_library" deviceset="CRYSTAL-8MHZ" device="HC49UP" value="8MHz"/>
+<part name="Z1" library="ExitControl_v2_master_library" deviceset="CRYSTAL-8MHZ" device="HC49UP" value="8MHz"/>
 <part name="CON5" library="pinhead" deviceset="PINHEAD_1X01" device="-2.54">
 <attribute name="BOM" value="EXCLUDE"/>
@@
 <attribute name="COLOR" value="BLUE"/>
 </part>
-<part name="R20" library="rc" deviceset="R" device="-0603" value="4K7"/>
+<part name="R20" library="rc" deviceset="R" device="-0603" value="4K7">
+<attribute name="ASSY" value="DNM"/>
+</part>
 <part name="+P1" library="supply_symbols" deviceset="3.3V" device=""/>
 <part name="+P26" library="supply_symbols" deviceset="5V" device=""/>
 <part name="CON7" library="pinhead" deviceset="PINHEAD_1X03" device="-2.54"/>
+<part name="R21" library="rc" deviceset="R" device="-R1206" value="24R"/>
+<part name="+P27" library="supply_symbols" deviceset="SUPPLY" device=""/>
+<part name="Q5" library="motion_detect_masterlib" deviceset="IRLML2502" device="-SOT23"/>
+<part name="GND38" library="supply_symbols" deviceset="GND" device="" value="GND"/>
+<part name="R22" library="rc" deviceset="R" device="-0603" value="4K7">
+<attribute name="ASSY" value="DNM"/>
+</part>
+<part name="+P28" library="supply_symbols" deviceset="3.3V" device=""/>
+<part name="R23" library="rc" deviceset="R" device="-0603" value="4K7"/>
+<part name="R24" library="rc" deviceset="R" device="-R1206" value="24R"/>
 </parts>
 <sheets>
@@
 <instance part="R17" gate="G$1" x="12.7" y="25.4" rot="R270"/>
 <instance part="GND22" gate="1" x="12.7" y="15.24"/>
-<instance part="SW1" gate="G$1" x="170.18" y="55.88" rot="R270"/>
-<instance part="GND7" gate="1" x="170.18" y="45.72"/>
+<instance part="SW1" gate="G$1" x="170.18" y="40.64" rot="R270"/>
+<instance part="GND7" gate="1" x="170.18" y="27.94"/>
 <instance part="GND37" gate="1" x="162.56" y="88.9"/>
 <instance part="R1" gate="G$1" x="45.72" y="137.16" rot="R270"/>
@@
 <instance part="+P23" gate="G$1" x="43.18" y="160.02" rot="R180"/>
 <instance part="R19" gate="G$1" x="99.06" y="60.96"/>
-<instance part="Z1_1" gate="G$1" x="73.66" y="99.06" rot="R180"/>
+<instance part="Z1" gate="G$1" x="73.66" y="99.06" rot="R180"/>
 <instance part="CON5" gate="G$1" x="203.2" y="157.48" rot="R180">
 <attribute name="BOM" x="203.2" y="157.48" size="1.27" layer="96" rot="R180" display="off"/>
@@
 <attribute name="COLOR" x="175.26" y="114.3" size="1.778" layer="96" display="off"/>
 </instance>
-<instance part="R20" gate="G$1" x="71.12" y="132.08" rot="R270"/>
+<instance part="R20" gate="G$1" x="71.12" y="132.08" rot="R270">
+<attribute name="ASSY" x="71.12" y="132.08" size="1.27" layer="96" rot="R270" display="off"/>
+</instance>
 <instance part="+P1" gate="G$1" x="71.12" y="139.7"/>
 <instance part="+P26" gate="G$1" x="25.4" y="127" rot="R270"/>
 <instance part="CON7" gate="G$1" x="248.92" y="147.32" rot="R180"/>
+<instance part="R21" gate="G$1" x="139.7" y="157.48" rot="R90"/>
+<instance part="+P27" gate="G$1" x="139.7" y="167.64"/>
+<instance part="Q5" gate="G$1" x="137.16" y="139.7"/>
+<instance part="GND38" gate="1" x="139.7" y="119.38"/>
+<instance part="R22" gate="G$1" x="175.26" y="55.88" rot="R270">
+<attribute name="ASSY" x="175.26" y="55.88" size="1.27" layer="96" rot="R270" display="off"/>
+</instance>
+<instance part="+P28" gate="G$1" x="175.26" y="66.04"/>
+<instance part="R23" gate="G$1" x="132.08" y="132.08" rot="R270"/>
+<instance part="R24" gate="G$1" x="134.62" y="157.48" rot="R90"/>
 </instances>
 <busses>
@@
 <pinref part="CON3" gate="G$1" pin="8"/>
 <pinref part="GND8" gate="1" pin="GND"/>
-<wire x1="15.24" y1="142.24" x2="22.86" y2="142.24" width="0.1524" layer="91"/>
+<wire x1="15.24" y1="142.24" x2="17.78" y2="142.24" width="0.1524" layer="91"/>
+<pinref part="CON3" gate="G$1" pin="7"/>
+<wire x1="17.78" y1="142.24" x2="22.86" y2="142.24" width="0.1524" layer="91"/>
+<wire x1="15.24" y1="139.7" x2="17.78" y2="139.7" width="0.1524" layer="91"/>
+<wire x1="17.78" y1="139.7" x2="17.78" y2="142.24" width="0.1524" layer="91"/>
+<junction x="17.78" y="142.24"/>
 </segment>
 <segment>
@@
 <pinref part="SW1" gate="G$1" pin="2"/>
 <pinref part="GND7" gate="1" pin="GND"/>
-<wire x1="170.18" y1="50.8" x2="170.18" y2="48.26" width="0.1524" layer="91"/>
+<wire x1="170.18" y1="35.56" x2="170.18" y2="30.48" width="0.1524" layer="91"/>
+</segment>
+<segment>
+<pinref part="GND38" gate="1" pin="GND"/>
+<pinref part="Q5" gate="G$1" pin="S"/>
+<wire x1="139.7" y1="121.92" x2="139.7" y2="124.46" width="0.1524" layer="91"/>
+<pinref part="R23" gate="G$1" pin="2"/>
+<wire x1="139.7" y1="124.46" x2="139.7" y2="137.16" width="0.1524" layer="91"/>
+<wire x1="132.08" y1="127" x2="132.08" y2="124.46" width="0.1524" layer="91"/>
+<wire x1="132.08" y1="124.46" x2="139.7" y2="124.46" width="0.1524" layer="91"/>
+<junction x="139.7" y="124.46"/>
 </segment>
 </net>
@@
 </segment>
 <segment>
-<pinref part="CON3" gate="G$1" pin="7"/>
-<wire x1="15.24" y1="139.7" x2="20.32" y2="139.7" width="0.1524" layer="91"/>
-<label x="20.32" y="139.7" size="1.27" layer="95" xref="yes"/>
+<pinref part="IC1" gate="G$1" pin="CE"/>
+<wire x1="114.3" y1="25.4" x2="111.76" y2="25.4" width="0.1524" layer="91"/>
+<label x="114.3" y="12.7" size="1.27" layer="95" font="vector" xref="yes"/>
+<wire x1="111.76" y1="25.4" x2="111.76" y2="12.7" width="0.1524" layer="91"/>
+<wire x1="111.76" y1="12.7" x2="114.3" y2="12.7" width="0.1524" layer="91"/>
 </segment>
 </net>
@@
 </segment>
 <segment>
-<pinref part="IC1" gate="G$1" pin="CE"/>
-<wire x1="114.3" y1="25.4" x2="111.76" y2="25.4" width="0.1524" layer="91"/>
-<label x="114.3" y="12.7" size="1.27" layer="95" font="vector" xref="yes"/>
-<wire x1="111.76" y1="25.4" x2="111.76" y2="12.7" width="0.1524" layer="91"/>
-<wire x1="111.76" y1="12.7" x2="114.3" y2="12.7" width="0.1524" layer="91"/>
+<pinref part="Q5" gate="G$1" pin="G"/>
+<wire x1="134.62" y1="139.7" x2="132.08" y2="139.7" width="0.1524" layer="91"/>
+<label x="129.54" y="139.7" size="1.27" layer="95" rot="R180" xref="yes"/>
+<pinref part="R23" gate="G$1" pin="1"/>
+<wire x1="132.08" y1="139.7" x2="129.54" y2="139.7" width="0.1524" layer="91"/>
+<wire x1="132.08" y1="137.16" x2="132.08" y2="139.7" width="0.1524" layer="91"/>
+<junction x="132.08" y="139.7"/>
 </segment>
 </net>
@@
 <wire x1="71.12" y1="137.16" x2="71.12" y2="139.7" width="0.1524" layer="91"/>
 </segment>
+<segment>
+<pinref part="R22" gate="G$1" pin="1"/>
+<pinref part="+P28" gate="G$1" pin="VDD_3V3"/>
+<wire x1="175.26" y1="66.04" x2="175.26" y2="60.96" width="0.1524" layer="91"/>
+</segment>
 </net>
 <net name="A5" class="0">
@@
 <pinref part="C12" gate="G$1" pin="1"/>
 <wire x1="68.58" y1="96.52" x2="68.58" y2="99.06" width="0.1524" layer="91"/>
-<pinref part="Z1_1" gate="G$1" pin="2"/>
+<pinref part="Z1" gate="G$1" pin="2"/>
 <wire x1="68.58" y1="99.06" x2="68.58" y2="111.76" width="0.1524" layer="91"/>
 <wire x1="71.12" y1="99.06" x2="68.58" y2="99.06" width="0.1524" layer="91"/>
@@
 <pinref part="C11" gate="G$1" pin="1"/>
 <wire x1="78.74" y1="96.52" x2="78.74" y2="99.06" width="0.1524" layer="91"/>
-<pinref part="Z1_1" gate="G$1" pin="1"/>
+<pinref part="Z1" gate="G$1" pin="1"/>
 <wire x1="78.74" y1="99.06" x2="78.74" y2="109.22" width="0.1524" layer="91"/>
 <wire x1="76.2" y1="99.06" x2="78.74" y2="99.06" width="0.1524" layer="91"/>
@@
 <wire x1="162.56" y1="116.84" x2="162.56" y2="124.46" width="0.1524" layer="91"/>
 </segment>
+<segment>
+<pinref part="R21" gate="G$1" pin="2"/>
+<pinref part="+P27" gate="G$1" pin="SUP"/>
+<wire x1="139.7" y1="167.64" x2="139.7" y2="165.1" width="0.1524" layer="91"/>
+<pinref part="R24" gate="G$1" pin="2"/>
+<wire x1="139.7" y1="165.1" x2="139.7" y2="162.56" width="0.1524" layer="91"/>
+<wire x1="134.62" y1="162.56" x2="134.62" y2="165.1" width="0.1524" layer="91"/>
+<wire x1="134.62" y1="165.1" x2="139.7" y2="165.1" width="0.1524" layer="91"/>
+<junction x="139.7" y="165.1"/>
+</segment>
 </net>
 <net name="N$13" class="0">
@@
 <segment>
 <pinref part="IC4" gate="G$1" pin="PD3"/>
+<label x="76.2" y="127" size="1.27" layer="95" rot="R180" xref="yes"/>
 <wire x1="76.2" y1="127" x2="81.28" y2="127" width="0.1524" layer="91"/>
-<label x="76.2" y="127" size="1.27" layer="95" rot="R180" xref="yes"/>
-</segment>
-<segment>
-<label x="170.18" y="68.58" size="1.27" layer="95" rot="R90" xref="yes"/>
+</segment>
+<segment>
+<label x="170.18" y="50.8" size="1.27" layer="95" rot="R90" xref="yes"/>
 <pinref part="SW1" gate="G$1" pin="1"/>
-<wire x1="170.18" y1="60.96" x2="170.18" y2="68.58" width="0.1524" layer="91"/>
+<wire x1="170.18" y1="45.72" x2="170.18" y2="48.26" width="0.1524" layer="91"/>
+<pinref part="R22" gate="G$1" pin="2"/>
+<wire x1="170.18" y1="48.26" x2="170.18" y2="50.8" width="0.1524" layer="91"/>
+<wire x1="175.26" y1="50.8" x2="175.26" y2="48.26" width="0.1524" layer="91"/>
+<wire x1="175.26" y1="48.26" x2="170.18" y2="48.26" width="0.1524" layer="91"/>
+<junction x="170.18" y="48.26"/>
 </segment>
 </net>
@@
 </segment>
 </net>
+<net name="N$26" class="0">
+<segment>
+<pinref part="R21" gate="G$1" pin="1"/>
+<pinref part="Q5" gate="G$1" pin="D"/>
+<wire x1="139.7" y1="147.32" x2="139.7" y2="149.86" width="0.1524" layer="91"/>
+<pinref part="R24" gate="G$1" pin="1"/>
+<wire x1="139.7" y1="149.86" x2="139.7" y2="152.4" width="0.1524" layer="91"/>
+<wire x1="134.62" y1="152.4" x2="134.62" y2="149.86" width="0.1524" layer="91"/>
+<wire x1="134.62" y1="149.86" x2="139.7" y2="149.86" width="0.1524" layer="91"/>
+<junction x="139.7" y="149.86"/>
+</segment>
+</net>
